Commit message: update XACRO

File: serpens_urdf_description/urdf/serpens_urdf.xacro (robot description, xacro)
@@ -586,5 +586,5 @@
   <child link="arm_servo_tool_1"/>
   <axis xyz="-0.0 0.0 -1.0"/>
-  <limit effort="100" lower="1.570796" upper="4.712389" velocity="100"/>
+  <limit effort="100" lower="-1.570796" upper="1.570796" velocity="100"/>
 </joint>
 <joint name="f15" type="fixed">

Commit message: delete some link

File: serpens_urdf_description/urdf/serpens_urdf.xacro (robot description, xacro)
@@ -5,9 +5,4 @@
 <xacro:include filename="$(find serpens_urdf_description)/urdf/serpens_urdf.gazebo" />
 <link name="base_link">
-  <inertial>
-    <origin rpy="0 0 0" xyz="0.00027997054451526365 -0.00019064006265276712 0.01910383815728144"/>
-    <mass value="0.20475393508704573"/>
-    <inertia ixx="0.000171" ixy="-0.0" ixz="1e-06" iyy="0.000189" iyz="-0.0" izz="0.000318"/>
-  </inertial>
   <visual>
     <origin rpy="0 0 0" xyz="0 0 0"/>
@@ -461,24 +456,4 @@
     <geometry>
       <mesh filename="package://serpens_urdf_description/meshes/link3_2_1.stl" scale="0.001 0.001 0.001"/>
-    </geometry>
-  </collision>
-</link>
-<link name="link2_pair_1">
-  <inertial>
-    <origin rpy="0 0 0" xyz="0.028812952511745295 0.002249900962215688 -0.017756131216635412"/>
-    <mass value="0.03005223787841536"/>
-    <inertia ixx="3e-06" ixy="-0.0" ixz="3e-06" iyy="1e-05" iyz="0.0" izz="7e-06"/>
-  </inertial>
-  <visual>
-    <origin rpy="0 0 0" xyz="0.068223 -0.023324 -0.1039"/>
-    <geometry>
-      <mesh filename="package://serpens_urdf_description/meshes/link2_pair_1.stl" scale="0.001 0.001 0.001"/>
-    </geometry>
-    <material name="silver"/>
-  </visual>
-  <collision>
-    <origin rpy="0 0 0" xyz="0.068223 -0.023324 -0.1039"/>
-    <geometry>
-      <mesh filename="package://serpens_urdf_description/meshes/link2_pair_1.stl" scale="0.001 0.001 0.001"/>
     </geometry>
   </collision>
@@ -608,8 +583,3 @@
   <child link="link3_2_1"/>
 </joint>
-<joint name="f19" type="fixed">
-  <origin rpy="0 0 0" xyz="0.0 0.033 0.0"/>
-  <parent link="link3_2_1"/>
-  <child link="link2_pair_1"/>
-</joint>
 </robot>
